Commit message: dolly ekleme çalışmaları

File: dolly.urdf.xacro (robot description, xacro)
@@ -12,5 +12,5 @@
       <origin rpy="0 0 0" xyz="0 0 0" />
       <geometry>
-        <mesh filename="package://simulation/meshes/Lowpolyhuman.dae"  scale="1 1 1" />
+        <mesh filename="package://home/beraa/ros2_ws/src/via_description/meshes/Lowpolyhuman.dae"  scale="1 1 1" />
       </geometry>
       <material name="Red"/>
@@ -19,5 +19,5 @@
       <origin rpy="0 0 0" xyz="0 0 0" />
       <geometry>
-        <mesh filename="package://simulation/meshes/Lowpolyhuman.dae" scale="1 1 1" />
+        <mesh filename="package://home/beraa/ros2_ws/src/via_description/meshes/Lowpolyhuman.dae" scale="1 1 1" />
       </geometry>
     </collision>
